Commit message: Primera prueba urdf con diseño dron
Se elimina tambien las carpetas de compilación pq faltaba el gitignore

File: ros_ws/src/chimuelo_bringup/urdf/prueba_chimuelo.urdf (robot description, URDF)
Before this commit: robot chimuelo_x500, 8 links, 7 joints
Links:
- link base_link: geometry collision box size=0.4 0.4 0.2; visual mesh filename=package://chimuelo_bringup/meshes/chimuelo.stl scale=0.001 0.001 0.001

Commit message: Urdf + STL del diseño cad

File: ros_ws/src/chimuelo_bringup/urdf/prueba_chimuelo.urdf (robot description, URDF)
Before this commit: robot chimuelo_x500, 8 links, 7 joints
Links:
- removed link arm_fl
- removed link arm_fr
- removed link arm_rl
- removed link arm_rr
- removed link landing_gear_left
- removed link landing_gear_right
- link base_link: geometry collision box size=0.5 0.5 0.25; visual mesh filename=package://chimuelo_bringup/meshes/chimuelo.stl scale=0.001 0.001 0.001
Joints:
- removed joint base_to_arm_fl
- removed joint base_to_arm_fr
- removed joint base_to_arm_rl
- removed joint base_to_arm_rr
- removed joint gear_left_joint
- removed joint gear_right_joint

Commit message: camera_link

File: ros_ws/src/chimuelo_bringup/urdf/prueba_chimuelo.urdf (robot description, URDF)
Before this commit: robot chimuelo_x500, 2 links, 1 joints
Joints:
- joint drone_camera_joint: origin xyz=0.15 0.0 -0.04 rpy=0 0 0 -> xyz=0.15 0.0 -0.04 rpy=0 0.24 0

Commit message: EKF File + Base_Footprint en URDF

File: ros_ws/src/chimuelo_bringup/urdf/prueba_chimuelo.urdf (robot description, URDF)
Before this commit: robot chimuelo_x500, 2 links, 1 joints
Links:
- added link base_footprint
Joints:
- added joint base_footprint_joint: type fixed, parent base_link, child base_footprint, origin xyz=0 0 -0.26 rpy=0 0 0

Commit message: Urdf actualizado
Se ha ajustado camera_link a nuestro robot real

File: ros_ws/src/chimuelo_bringup/urdf/prueba_chimuelo.urdf (robot description, URDF)
Before this commit: robot chimuelo_x500, 3 links, 2 joints
Joints:
- joint drone_camera_joint: origin xyz=0.15 0.0 -0.04 rpy=0 0.24 0 -> xyz=0.18 0.0 -0.045 rpy=0 0 0
